File: board.kicad_pcb (KiCad board)
At the start: 4 copper layers, 92 parts, among them J1 GT-USB-7010ASV, J2 Battery, J3 Speaker, J4 SWD, SW1 Button L, SW2 Button R, SW3 Menu, U1 RP2040, U2 BQ24074RGT, U3 RT6160A, U4 VDD331MCTA, U5 W25Q128JVPIQ, U6 USBLC6-2SC6, U7 TPS22914BYFPR, U8 MAX98357AEWL, U9 MT3608B, Y1 ABM8-272-T3

Commit message: 'yay'
Parts:
- removed the C8 at (174.6, 46.0)
- removed the J3 at (218.1, 77.8)
- removed JP1: BOOTSEL, Jumper:SolderJumper-2_P1.3mm_Open_Pad1.0x1.5mm
- removed JP2: RESET, Jumper:SolderJumper-2_P1.3mm_Open_Pad1.0x1.5mm
- removed the PL1 at (95.4, 86.7)
- removed the R20 at (136.7, 73.3)
- removed the R5 at (199.3, 39.9)
- removed REF**: OLED-128O064D, Display:OLED-128O064D
- removed REF**: OLED 128x64 0.96", Custom:OLED_128x64_0.96in_30P
- removed the TP1 at (212.0, 63.5)
- removed the U7 at (199.3, 38.9)
- added C1: 100nF, Capacitor_SMD:C_0201_0603Metric, B.Cu at (70.4, 27.2)
- added D1: LED_BUTTON_L, PCM_marbastlib-mx:LED_MX_6028R, B.Cu at (29.7, 34.8)
- added D2: LED_BUTTON_R, PCM_marbastlib-mx:LED_MX_6028R, B.Cu at (96.3, 34.8)
- added J4: Speaker, Connector_PinHeader_2.54mm:PinHeader_1x02_P2.54mm_Vertical, F.Cu at (42.7, 37.6)
- added R12: 27, Resistor_SMD:R_0201_0603Metric, B.Cu at (75.5, 34.2)
- added R19: 140k, Resistor_SMD:R_0201_0603Metric, B.Cu at (87.8, 34.9)
- added R21: 5.1k, Resistor_SMD:R_0201_0603Metric, B.Cu at (60.0, 28.9)
- added R22: 140k, Resistor_SMD:R_0201_0603Metric, B.Cu at (55.9, 28.9)
- added TP10: BOOTSEL, TestPoint:TestPoint_Pad_1.0x1.0mm, B.Cu at (79.7, 17.9)
- added TP11: RESET, TestPoint:TestPoint_Pad_1.0x1.0mm, B.Cu at (68.1, 43.0)
- added U9: MT9700-N, Package_TO_SOT_SMD:SOT-23-5, B.Cu at (58.0, 30.0)
- C22: renamed from C29; moved to B.Cu
- C23: renamed from C38; moved to B.Cu
- C24: renamed from C33; moved to B.Cu
- C25: renamed from C39; moved to B.Cu
- C26: renamed from C37; moved to B.Cu
- C31: renamed from C40; moved to B.Cu
- C32: renamed from C41; footprint Capacitor_SMD:C_0402_1005Metric -> Capacitor_SMD:C_0201_0603Metric; moved to B.Cu
- C35: renamed from C42; moved to B.Cu
- D3: renamed from D1; moved to B.Cu
- DS1: renamed from DS2; moved to B.Cu
- J1: value GT-USB-7010ASV -> UJ20-C-H-G-MSMT-6-P16-TR; footprint Connector_USB:USB_C_Receptacle_G-Switch_GT-USB-7010ASV -> footprints:SAMESKY_UJ20-C-H-G-MSMT-6-P16-TR
- J2: footprint Connector_PinHeader_1.27mm:PinHeader_1x02_P1.27mm_Vertical -> Connector_JST:JST_PH_B2B-PH-K_1x02_P2.00mm_Vertical
- L2: moved to B.Cu
- R10: renamed from R4; value 3.6k -> 5.1k
- R13: renamed from R6; moved to B.Cu
- R14: renamed from R12; moved to B.Cu
- R16: renamed from R13; footprint Resistor_SMD:R_0402_1005Metric -> Resistor_SMD:R_0201_0603Metric; moved to B.Cu
- R17: renamed from R19; value 10k -> 5.1k
- R18: value 3.6k -> 10k
- R20: renamed from R21; footprint Resistor_SMD:R_0402_1005Metric -> Resistor_SMD:R_0201_0603Metric; moved to B.Cu
- SW1, SW2: footprint Button_Switch_Keyboard:SW_Cherry_MX_1.00u_PCB -> PCM_Switch_Keyboard_Hotswap_Kailh:SW_Hotswap_Kailh_MX_Plated
- SW3: value Menu -> CK_KMS2xxGP; footprint Button_Switch_SMD:SW_Push_1P1T-MP_NO_Horizontal_Alps_SKRTLAE010 -> Button_Switch_SMD:SW_SPST_CK_KMS2xxGP
- TP1: renamed from TP2; footprint TestPoint:TestPoint_Pad_D2.0mm -> TestPoint:TestPoint_Pad_1.0x1.0mm
- TP2: renamed from TP3; footprint TestPoint:TestPoint_Pad_D2.0mm -> TestPoint:TestPoint_Pad_1.0x1.0mm
- TP3: renamed from TP4; footprint TestPoint:TestPoint_Pad_D2.0mm -> TestPoint:TestPoint_Pad_1.0x1.0mm
- TP4: renamed from TP10; footprint TestPoint:TestPoint_Pad_D2.0mm -> TestPoint:TestPoint_Pad_1.0x1.0mm
- TP5: renamed from TP9; footprint TestPoint:TestPoint_Pad_D2.0mm -> TestPoint:TestPoint_Pad_1.0x1.0mm
- TP6: renamed from TP7; footprint TestPoint:TestPoint_Pad_D2.0mm -> TestPoint:TestPoint_Pad_1.0x1.0mm
- TP7: renamed from TP5; footprint TestPoint:TestPoint_Pad_D2.0mm -> TestPoint:TestPoint_Pad_1.0x1.0mm
- TP8: value SNS_VBAT -> PWR_VSYS; footprint TestPoint:TestPoint_Pad_D2.0mm -> TestPoint:TestPoint_Pad_1.0x1.0mm
- TP9: renamed from TP6; footprint TestPoint:TestPoint_Pad_D2.0mm -> TestPoint:TestPoint_Pad_1.0x1.0mm; moved to B.Cu
- U3: renamed from U5; footprint Package_SO:SOIC-8_5.3x5.3mm_P1.27mm -> Package_SON:WSON-8-1EP_6x5mm_P1.27mm_EP3.4x4.3mm
- U7: renamed from U9; moved to B.Cu
- moved NT1 194.9 mm to (50.8, 33.1)
- moved TP7 182.2 mm to (46.6, 42.7)
- moved TP3 181.6 mm to (45.0, 6.50)
- moved TP4 180.9 mm to (52.3, 11.0)
- moved TP5 177.8 mm to (52.8, 15.9)
- moved C34 177.0 mm to (48.8, 36.8)
- moved U8 175.4 mm to (50.6, 37.4)
- moved TP2 175.0 mm to (50.7, 6.10)
- moved R17 171.6 mm to (65.8, 32.4)
- moved R18 171.3 mm to (65.8, 31.7), turned to 0 degrees
- moved C33 168.8 mm to (54.3, 35.6)
- moved TP6 168.7 mm to (52.8, 41.6)
- moved TP8 160.2 mm to (68.2, 16.5)
- moved J2 159.8 mm to (42.9, 22.2), turned to 0 degrees
- moved R5 159.0 mm to (75.9, 32.5), turned to 0 degrees
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- renumbered C17 to C10, C18 to C11, C20 to C12, C21 to C13, C19 to C14, C23 to C15, C24 to C16, C34 to C17, C2 to C18, C22 to C19, C16 to C2, C3 to C20, C1 to C21, C4 to C27, C5 to C28, C7 to C29, C15 to C3, C6 to C30, C35 to C33, C36 to C34, C14 to C4, C13 to C5, C12 to C6, C11 to C7, C10 to C8, J4 to J3, R9 to R1, R3 to R11, R1 to R3, R15 to R4, R16 to R5, R10 to R6, R11 to R7, R7 to R8, R8 to R9, U6 to U1, U1 to U2, U2 to U4, U4 to U5, U3 to U6
Connections:
- net /PERIPHERAL_ON renamed /DISP_REG_EN
- net /SNS_VBAT renamed /PWR_VSYS
- net /SNS_~{CHG} renamed /PWR_~{CHG}
- net /SNS_~{PGOOD} renamed /PWR_~{PGOOD}
- J2 pad 1: VBAT -> GND
- J2 pad 2: GND -> VBAT
- NT1 pad 1: Net-(U3-AGND) -> Net-(U6-AGND)
- R17 pad 2: VBAT_GATED -> VSYS_GATED
- U2 pad 11: /AUDIO_I2S_LRCK -> unconnected-(U2-GPIO8-Pad11)
- U2 pad 12: /AUDIO_I2S_SD -> unconnected-(U2-GPIO9-Pad12)
- U2 pad 29: unconnected-(U1-GPIO18-Pad29) -> /AUDIO_I2S_LRCK
- U2 pad 30: unconnected-(U1-GPIO19-Pad30) -> /AUDIO_I2S_BCLK
- U2 pad 31: unconnected-(U1-GPIO20-Pad31) -> /AUDIO_I2S_DOUT
- U2 pad 32: unconnected-(U1-GPIO21-Pad32) -> /AUDIO_I2S_SD
- U2 pad 34: unconnected-(U1-GPIO22-Pad34) -> /PWR_CHG_EN
- U2 pad 35: unconnected-(U1-GPIO23-Pad35) -> /PWR_PERIPH_EN
- U2 pad 8: /AUDIO_I2S_DOUT -> /LED_DIN
- U2 pad 9: /AUDIO_I2S_BCLK -> unconnected-(U2-GPIO7-Pad9)
- U4 pad 4: GND -> /PWR_CHG_EN
- U6 pad B1: Net-(U3-AGND) -> Net-(U6-AGND)
- U6 pad C1: Net-(U3-AGND) -> Net-(U6-AGND)
- U6 pad D1: Net-(U3-AGND) -> unconnected-(U6-SCL-PadD1)
- U6 pad E1: Net-(U3-AGND) -> unconnected-(U6-SDA-PadE1)
Routing:
- net VSYS_GATED: track 0.00 -> 79.1 mm, vias 0 -> 4
- net Net-(D1-DIN): track 0.00 -> 66.4 mm, vias 0 -> 2
- net VSYS: track 0.00 -> 59.6 mm, vias 0 -> 16
- net /BUTTON_L: track 0.00 -> 58.8 mm, vias 0 -> 2
- net GND: track 0.00 -> 44.1 mm, vias 0 -> 44
- net /BUTTON_MENU: track 0.00 -> 32.1 mm, vias 0 -> 4
- net 3V3: track 0.05 -> 29.8 mm, vias 0 -> 18
- net Net-(D2-DIN): track 0.00 -> 29.2 mm, vias 0 -> 2
- net /BUTTON_R: track 0.00 -> 26.6 mm, vias 0 -> 2
- net /PWR_CHG_EN: track 0.00 -> 23.4 mm, vias 0 -> 2
- net /PWR_~{PGOOD}: track 0.00 -> 22.8 mm, vias 0 -> 2
- net /DISP_REG_EN: track 0.00 -> 22.2 mm
- net VBUS: track 0.00 -> 22.1 mm, vias 0 -> 3
- net /PWR_~{CHG}: track 0.00 -> 20.3 mm, vias 0 -> 2
- net /AUDIO_I2S_LRCK: track 0.00 -> 19.6 mm
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- added copper zone on In1.Cu, net VSYS
Other:
- board outline added: 86 x 19.4 mm
- board text removed: "https://ydlbattery.com/products/ydl-3-7v-750mah-782240-rechargeable-lipo-battery-with-jst-connector#/ thick: 8mm width: 22mm height: 42mm"

Commit message: wip
Parts:
- TP8: value PWR_VSYS -> SNS_VBAT
- U3: value W25Q128JVPIQ -> W25Q128JVSIQ; footprint Package_SON:WSON-8-1EP_6x5mm_P1.27mm_EP3.4x4.3mm -> Package_SO:SOIC-8_5.3x5.3mm_P1.27mm
- moved J3 42.3 mm to (63.0, 50.5), turned to 90 degrees
- moved C16 26.8 mm to (53.4, 37.1), turned to 90 degrees
- moved SW3 24.7 mm to (76.5, 21.4)
- moved Y1 21.9 mm to (55.8, 37.1), turned to 0 degrees
- moved R1 16.8 mm to (58.4, 36.3), turned to 90 degrees
- moved C15 16.7 mm to (58.4, 38.0), turned to -90 degrees
- moved R8 14.9 mm to (69.4, 33.2), turned to 0 degrees
- moved C2 14.1 mm to (56.7, 34.9), turned to 180 degrees
- moved R9 13.9 mm to (69.4, 32.5), turned to 0 degrees
- moved C14 13.6 mm to (56.7, 34.1), turned to 180 degrees
- moved U1 11.7 mm to (71.8, 22.2)
- moved TP8 11.3 mm to (60.8, 8.05)
- moved C7 9.31 mm to (66.6, 37.9)
- moved R12 9.31 mm to (66.6, 37.1)
- moved R5 8.82 mm to (68.0, 36.5)
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Connections:
- net /PWR_VSYS renamed /PWR_VBAT
Routing:
- net VSYS_GATED: track 79.1 -> 0.00 mm, vias 4 -> 0
- net Net-(D1-DIN): track 66.4 -> 0.00 mm, vias 2 -> 0
- net VSYS: track 59.6 -> 0.04 mm, vias 16 -> 0
- net /BUTTON_L: track 58.8 -> 0.65 mm, vias 2 -> 0
- net Net-(D2-DIN): track 29.2 -> 0.00 mm, vias 2 -> 0
- net /BUTTON_MENU: track 32.1 -> 4.10 mm, vias 4 -> 2
- net /BUTTON_R: track 26.6 -> 0.00 mm, vias 2 -> 0
- net /PWR_CHG_EN: track 23.4 -> 0.00 mm, vias 2 -> 0
- net /PWR_~{PGOOD}: track 22.8 -> 0.00 mm, vias 2 -> 0
- net /DISP_REG_EN: track 22.2 -> 0.00 mm
- net /PWR_~{CHG}: track 20.3 -> 0.00 mm, vias 2 -> 0
- net /AUDIO_I2S_LRCK: track 19.6 -> 0.00 mm
- net /PWR_PERIPH_EN: track 17.8 -> 0.00 mm, vias 2 -> 0
- net /AUDIO_I2S_BCLK: track 17.1 -> 0.00 mm
- net /AUDIO_I2S_SD: track 17.1 -> 0.00 mm
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- removed copper zone on In1.Cu, net VSYS
Other:
- outline, holes or cut-outs redrawn

Commit message: wip
Parts:
- moved TP10 9.10 mm to (69.4, 16.2)
- moved TP1 2.93 mm to (66.6, 16.2)
- moved R5 0.96 mm to (67.0, 36.5), turned to -45 degrees
- moved C7 0.85 mm to (65.8, 37.9), turned to -45 degrees
- moved R4 0.54 mm to (67.5, 36.0), turned to 135 degrees
- moved R12 0.37 mm to (66.3, 37.3), turned to 135 degrees
- moved R18 0.10 mm to (60.8, 29.1)
- moved R17 0.10 mm to (60.3, 29.6)
- moved C4 0.07 mm to (58.9, 31.0)
Routing:
- net /DISP_PIN_DC: track 0.00 -> 24.0 mm
- net /DISP_PIN_MOSI: track 0.00 -> 23.0 mm, vias 0 -> 2
- net /DISP_PIN_SCLK: track 0.00 -> 21.8 mm
- net /DISP_PIN_RST: track 0.00 -> 21.4 mm, vias 0 -> 2
- net /DISP_PIN_CS: track 1.83 -> 21.4 mm, vias 0 -> 2
- net GND: track 32.0 -> 47.2 mm, vias 13 -> 32
- net 9V: track 2.82 -> 10.5 mm
- net 1V1: track 17.8 -> 24.3 mm
- net VSYS: track 0.04 -> 5.09 mm, vias 0 -> 10
- net VBAT: track 1.21 -> 5.04 mm
- net Net-(D3-A): track 0.00 -> 3.28 mm
- net Net-(L1-Pad2): track 0.00 -> 2.13 mm
- net Net-(L1-Pad1): track 0.00 -> 2.13 mm
- net Net-(U7-FB): track 0.00 -> 2.09 mm
- net Net-(U4-ISET): track 0.00 -> 1.90 mm
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- added copper zone on In1.Cu, net VSYS

Commit message: routing complete??
Parts:
- moved C33 4.12 mm to (50.2, 34.6), turned to 0 degrees
- moved U8 2.77 mm to (49.9, 37.0)
- moved C34 2.72 mm to (49.6, 35.7)
- moved C28 0.70 mm to (51.0, 26.8)
- moved C29 0.70 mm to (50.2, 32.6)
- moved C30 0.70 mm to (50.2, 31.1)
- moved R10 0.70 mm to (48.6, 25.1)
- moved R22 0.70 mm to (56.0, 30.1)
- moved U4 0.70 mm to (51.4, 23.4)
- moved C17 0.70 mm to (54.3, 25.5)
- moved C18 0.70 mm to (53.0, 25.8)
- moved C20 0.70 mm to (54.3, 22.5)
- moved C21 0.70 mm to (48.6, 22.5)
- moved C27 0.70 mm to (49.0, 26.8)
- moved L1 0.70 mm to (49.5, 29.0)
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Connections:
- U2 pad 34: /PWR_CHG_EN -> /PWR_PERIPH_EN
- U2 pad 35: /PWR_PERIPH_EN -> /PWR_CHG_EN
Routing:
- net VSYS_GATED: track 0.00 -> 91.4 mm, vias 0 -> 4
- net Net-(D1-DIN): track 0.00 -> 65.3 mm, vias 0 -> 2
- net /BUTTON_L: track 0.65 -> 44.9 mm, vias 0 -> 1
- net Net-(D2-DIN): track 0.00 -> 37.9 mm, vias 0 -> 2
- net /BUTTON_R: track 0.00 -> 36.8 mm, vias 0 -> 1
- net VSYS: track 5.09 -> 39.0 mm, vias 10 -> 14
- net /BUTTON_MENU: track 4.10 -> 28.0 mm, vias 2 -> 3
- net /DISP_REG_EN: track 1.34 -> 24.1 mm, vias 0 -> 2
- net /PWR_CHG_EN: track 0.64 -> 17.0 mm, vias 1 -> 2
- net /PWR_~{CHG}: track 0.87 -> 15.9 mm, vias 1 -> 2
- net /PWR_~{PGOOD}: track 0.76 -> 15.4 mm, vias 1 -> 2
- net /AUDIO_I2S_LRCK: track 0.00 -> 12.9 mm, vias 0 -> 2
- net /AUDIO_I2S_SD: track 0.00 -> 12.3 mm, vias 0 -> 2
- net /AUDIO_I2S_DOUT: track 0.00 -> 11.6 mm, vias 0 -> 2
- net /AUDIO_I2S_BCLK: track 0.00 -> 11.5 mm, vias 0 -> 2
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Other:
- outline, holes or cut-outs redrawn

Commit message: wip
Parts:
- removed J3: SWD, Connector_PinHeader_2.54mm:PinHeader_1x03_P2.54mm_Vertical
- removed PL1: Panel Footprint, Custom:OLED_128x64_1.3in_13P
- removed TP1: VBUS, TestPoint:TestPoint_Pad_1.0x1.0mm
- removed TP10: BOOTSEL, TestPoint:TestPoint_Pad_1.0x1.0mm
- removed TP11: RESET, TestPoint:TestPoint_Pad_1.0x1.0mm
- removed TP2: VSYS, TestPoint:TestPoint_Pad_1.0x1.0mm
- removed TP3: VBAT, TestPoint:TestPoint_Pad_1.0x1.0mm
- removed TP4: SNS_~{PGOOD}, TestPoint:TestPoint_Pad_1.0x1.0mm
- removed TP5: SNS_~{CHG}, TestPoint:TestPoint_Pad_1.0x1.0mm
- removed TP6: REG_EN, TestPoint:TestPoint_Pad_1.0x1.0mm
- removed TP7: 3V3, TestPoint:TestPoint_Pad_1.0x1.0mm
- removed TP8: SNS_VBAT, TestPoint:TestPoint_Pad_1.0x1.0mm
- removed TP9: 9V, TestPoint:TestPoint_Pad_1.0x1.0mm
- added R15: 1k, Resistor_SMD:R_0201_0603Metric, B.Cu at (55.7, 24.6)
- J4: footprint Connector_PinHeader_2.54mm:PinHeader_1x02_P2.54mm_Vertical -> Connector_JST:JST_GH_BM02B-GHS-TBT_1x02-1MP_P1.25mm_Vertical
- L1: value 0.47uH -> AFE201610SR47MBT
- U5: footprint Package_TO_SOT_SMD:SOT-23-3 -> Package_TO_SOT_SMD:SOT-23
- moved J4 1.57 mm to (43.8, 36.6), turned to 180 degrees
- moved C15 1.02 mm to (57.4, 38.0)
- moved R1 1.02 mm to (57.4, 36.3)
- moved C16 0.85 mm to (52.5, 37.1)
- moved Y1 0.85 mm to (55.0, 37.1)
- moved L1 0.69 mm to (48.9, 29.0)
- moved C7 0.25 mm to (65.7, 37.9)
- moved R12 0.21 mm to (66.2, 37.4)
Connections:
- net /AUDIO_I2S_SD renamed /AUDIO_I2S_EN
- U2 pad 24: Net-(J3-Pin_1) -> unconnected-(U2-SWCLK-Pad24)
- U2 pad 25: Net-(J3-Pin_3) -> unconnected-(U2-SWD-Pad25)
- U4 pad 12: unconnected-(U4-ILIM-Pad12) -> Net-(U4-ILIM)
- U5 pad 1: GND -> REG_EN
- U5 pad 2: REG_EN -> GND
Routing:
- net GND: track 56.8 -> 67.5 mm, vias 40 -> 44
- net /BUTTON_L: track 44.9 -> 52.0 mm, vias 1 -> 2
- net VSYS: track 39.0 -> 42.0 mm
- net 3V3: track 34.3 -> 37.2 mm
- net /BUTTON_R: track 36.8 -> 39.8 mm, vias 1 -> 2
- net Net-(U4-ILIM): track 0.00 -> 2.86 mm
- net REG_EN: track 1.69 -> 2.93 mm
- net /XOUT: track 2.66 -> 3.68 mm
- net /DISP_PIN_CS: track 21.4 -> 22.4 mm
- net Net-(L1-Pad2): track 2.13 -> 3.07 mm
- net Net-(L1-Pad1): track 2.13 -> 3.02 mm
- net /XIN: track 4.65 -> 5.50 mm
- net VBUS: track 24.2 -> 23.5 mm

Commit message: done (?)
Parts:
- added TP1: GND, TestPoint:TestPoint_Pad_1.0x1.0mm, B.Cu at (40.0, 29.8)
- added TP2: RESET, TestPoint:TestPoint_Pad_1.0x1.0mm, B.Cu at (40.0, 27.8)
- added TP3: BOOTSEL, TestPoint:TestPoint_Pad_1.0x1.0mm, B.Cu at (40.0, 31.8)
- J3: renamed from J4; footprint Connector_JST:JST_GH_BM02B-GHS-TBT_1x02-1MP_P1.25mm_Vertical -> Connector_JST:JST_ZH_B2B-ZR_1x02_P1.50mm_Vertical
- moved C31 17.5 mm to (70.8, 36.1), turned to 0 degrees
- moved R17 15.9 mm to (71.7, 37.9), turned to 0 degrees
- moved C32 15.8 mm to (71.7, 37.2), turned to 0 degrees
- moved U8 10.3 mm to (74.4, 37.0), turned to 180 degrees
- moved R22 6.06 mm to (77.1, 33.5), turned to -90 degrees
- moved R13 5.67 mm to (60.6, 38.3), turned to 0 degrees
- moved L2 3.98 mm to (77.9, 37.9), turned to 180 degrees
- moved R21 3.61 mm to (78.2, 33.9), turned to 0 degrees
- moved D3 1.85 mm to (78.1, 36.2), turned to 180 degrees
- moved C35 1.77 mm to (80.5, 37.0), turned to -90 degrees
- moved J3 0.96 mm to (44.6, 37.0)
- moved J2 0.71 mm to (43.0, 22.9)
- renumbered R15 to R10, R10 to R11, R11 to R12, R12 to R13, R13 to R14, R14 to R15, R22 to R16, R16 to R17, R21 to R18, R17 to R19, R18 to R20, R19 to R21, R20 to R22, U9 to U7, U7 to U8, U8 to U9
Connections:
- D1 pad 2: unconnected-(D1-DOUT-Pad2) -> Net-(D1-DOUT)
- D2 pad 2: Net-(D1-DIN) -> unconnected-(D2-DOUT-Pad2)
- D2 pad 3: Net-(D2-DIN) -> Net-(D1-DOUT)
- R13 pad 1: Net-(D2-DIN) -> Net-(D1-DIN)
- U2 pad 16: unconnected-(U2-GPIO13-Pad16) -> /LED_DIN
- U2 pad 8: /LED_DIN -> unconnected-(U2-GPIO6-Pad8)
Routing:
- net Net-(D1-DOUT): track 0.00 -> 83.8 mm, vias 0 -> 2
- net Net-(D2-DIN): track 37.7 -> 0.00 mm, vias 2 -> 0
- net Net-(R9-Pad1): track 0.00 -> 35.3 mm, vias 0 -> 2
- net Net-(D1-DIN): track 65.3 -> 30.5 mm
- net Net-(U2-RUN): track 0.00 -> 26.9 mm, vias 0 -> 2
- net /DISP_REG_EN: track 24.1 -> 9.11 mm, vias 2 -> 0
- net GND: track 67.5 -> 76.8 mm, vias 44 -> 62
- net VSYS: track 42.0 -> 35.5 mm
- net VSYS_GATED: track 91.4 -> 97.4 mm
- net Net-(U8-FB): track 2.30 -> 7.43 mm
- net /DISP_PIN_RST: track 21.6 -> 17.0 mm
- net /DISP_PIN_CS: track 22.4 -> 18.1 mm
- net /DISP_PIN_SCLK: track 21.8 -> 17.9 mm, vias 0 -> 2
- net /DISP_PIN_MOSI: track 23.0 -> 19.2 mm
- net Net-(J3-Pin_2): track 4.58 -> 7.90 mm
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Other:
- outline, holes or cut-outs redrawn

Commit message: ordered
Parts:
- L2: value 4.7uH -> CMH160808B4R7MT
Routing:
- net 3V3: track 34.4 -> 34.5 mm, vias 19 -> 20
- added copper zone on In1.Cu, net GND
