File: board.kicad_sch (KiCad schematic)
At the start: 83 parts, among them J1 UJ20-C-H-G-MSMT-6-P16-TR, J2 Battery, J3 Speaker, SW1 Button L, SW2 Button R, SW3 CK_KMS2xxGP, U1 USBLC6-2SC6, U2 RP2040, U3 W25Q128JVSIQ, U4 BQ24074RGT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

Commit message: yay
Parts:
- J2: DigiKey (none) -> 455-1704-ND
- J3: DigiKey (none) -> 455-B2B-ZR-ND; Digikey 455-B2B-ZR-ND -> (none)
Changed lines of the file:
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@@
 			)
 		)
+		(property "DigiKey" "455-1704-ND"
+			(at 72.39 27.94 0)
+			(effects
+				(font
+					(size 1.27 1.27)
+				)
+				(hide yes)
+			)
+		)
 		(pin "1"
 		)
@@
 			)
 		)
-		(property "Digikey" "455-B2B-ZR-ND"
+		(property "Digikey" ""
+			(at 276.86 81.28 0)
+			(effects
+				(font
+					(size 1.27 1.27)
+				)
+				(hide yes)
+			)
+		)
+		(property "DigiKey" "455-B2B-ZR-ND"
 			(at 276.86 81.28 0)
 			(effects
